Commit message: Adjust FT sensor simulation
added floor

File: ur3_description/urdf/ur3e/ur3e.urdf.xacro (robot description, xacro)
@@ -296,5 +296,5 @@
     <link name="${prefix}tool0"/>
     <joint name="${prefix}wrist_3_link-tool0_fixed_joint" type="fixed">
-      <origin xyz="0 ${wrist_3_length} 0" rpy="${pi/-2.0} 0 0"/>
+      <origin xyz="0 ${wrist_3_length} 0" rpy="${pi/-2.0} 0 ${pi}"/>
       <parent link="${prefix}wrist_3_link"/>
       <child link="${prefix}tool0"/>

File: ur3_description/urdf/ur3e/ur3e_peg_gripper.urdf.xacro (robot description, xacro)
@@ -23,5 +23,5 @@
   </link>
   <joint name="robotiq_coupler_joint" type="fixed">
-    <origin xyz="0 0 0" rpy="${-pi/2.0} 0 0" />
+    <origin xyz="0 0 0" rpy="${pi/2.0} 0 0" />
     <parent link="tool0"/>
     <child link="robotiq_coupler"/>
@@ -49,5 +49,5 @@
   <gazebo>
     <plugin name="ft_sensor" filename="libgazebo_ros_ft_sensor.so">
-      <updateRate>100.0</updateRate>
+      <updateRate>500.0</updateRate>
       <topicName>ft_sensor/raw</topicName>
       <gaussianNoise>0.0</gaussianNoise>

Commit message: support beta driver
fix FT sensor again

File: ur3_description/urdf/ur3e/ur3e.urdf.xacro (robot description, xacro)
@@ -296,5 +296,5 @@
     <link name="${prefix}tool0"/>
     <joint name="${prefix}wrist_3_link-tool0_fixed_joint" type="fixed">
-      <origin xyz="0 ${wrist_3_length} 0" rpy="${pi/-2.0} 0 ${pi}"/>
+      <origin xyz="0 ${wrist_3_length} 0" rpy="${pi/-2.0} 0 0"/>
       <parent link="${prefix}wrist_3_link"/>
       <child link="${prefix}tool0"/>

File: ur3_description/urdf/ur3e/ur3e_peg_gripper.urdf.xacro (robot description, xacro)
@@ -23,5 +23,5 @@
   </link>
   <joint name="robotiq_coupler_joint" type="fixed">
-    <origin xyz="0 0 0" rpy="${pi/2.0} 0 0" />
+    <origin xyz="0 0 0" rpy="${-pi/2.0} 0 0" />
     <parent link="tool0"/>
     <child link="robotiq_coupler"/>

Commit message: bulk update
- Improve cartesian motion using either IKFast or Trac-Ik solvers
- Improve controller (arm) robustness to unexpected errors
- add tele-operation with a navigational 6d mouse

File: ur3_description/urdf/ur3e/ur3e.urdf.xacro (robot description, xacro)
@@ -280,4 +280,5 @@
     <xacro:unless value="$(arg use_effort_interface)">
       <xacro:ur_arm_transmission prefix="${prefix}" joint_interface="PositionJointInterface" />
+      <!-- <xacro:ur_arm_transmission prefix="${prefix}" joint_interface="VelocityJointInterface" /> -->
     </xacro:unless>
     <xacro:ur_arm_gazebo prefix="${prefix}" />

File: ur_pykdl/urdf/ur3e_robot.urdf (robot description, URDF)
Before this commit: robot ur3e, 11 links, 10 joints
Joints:
- joint shoulder_lift_joint: limit lower=-6.28318530718 upper=6.28318530718 effort=330.0 velocity=3.14 -> lower=-3.14159265359 upper=3.14159265359 effort=330.0 velocity=3.14
- joint shoulder_pan_joint: limit lower=-6.28318530718 upper=6.28318530718 effort=330.0 velocity=3.14 -> lower=-3.14159265359 upper=3.14159265359 effort=330.0 velocity=3.14
- joint wrist_1_joint: limit lower=-6.28318530718 upper=6.28318530718 effort=54.0 velocity=6.28 -> lower=-3.14159265359 upper=3.14159265359 effort=54.0 velocity=6.28
- joint wrist_2_joint: limit lower=-6.28318530718 upper=6.28318530718 effort=54.0 velocity=6.28 -> lower=-3.14159265359 upper=3.14159265359 effort=54.0 velocity=6.28
- joint wrist_3_joint: limit lower=-6.28318530718 upper=6.28318530718 effort=54.0 velocity=6.28 -> lower=-3.14159265359 upper=3.14159265359 effort=54.0 velocity=6.28
