Commit message: Fix Force/Torque sensor Gazebo

File: ur3_gazebo/urdf/ur_e_with_gripper.xacro (robot description, xacro)
@@ -103,18 +103,21 @@
   </gazebo>
   <!-- Equivalent to the OpenRAVE manipulator denso_robotiq_hande_gripper -->
-  <link name="ur3_robotiq_hande_gripper" />
+  <link name="ur_gripper_tip_link" />
   <joint name="manipulator_dummy_joint" type="fixed">
     <origin xyz="0 0 0.1441" rpy="0 0 0" />
     <parent link="robotiq_coupler"/>
-    <child link="ur3_robotiq_hande_gripper"/>
+    <child link="ur_gripper_tip_link"/>
   </joint>
   <!-- Attach the robotiq hand-e gripper -->
   <xacro:robotiq_hande_gripper prefix="" parent="robotiq_coupler" >
-    <origin xyz="0 0 0.004" rpy="0 0 ${pi/2}"/>
+    <origin xyz="0 0 0.004" rpy="0 0 ${-pi/2}"/>
   </xacro:robotiq_hande_gripper>
-  <!-- Gazebo FT sensor plugin -->
-  <gazebo reference="wrist_3_link-tool0_fixed_joint">
+  <!-- Gazebo Force/Torque sensor plugin -->
+  <gazebo reference="wrist_3_joint">
     <provideFeedback>true</provideFeedback>
   </gazebo>
+  <!-- <gazebo reference="wrist_3_joint">
+    <preserveFixedJoint>true</preserveFixedJoint>
+  </gazebo> -->
   <gazebo>
     <plugin name="ft_sensor" filename="libgazebo_ros_ft_sensor.so">
@@ -122,5 +125,5 @@
       <topicName>ft_sensor/raw</topicName>
       <gaussianNoise>0.0</gaussianNoise>
-      <jointName>wrist_3_link-tool0_fixed_joint</jointName>
+      <jointName>wrist_3_joint</jointName>
     </plugin>
   </gazebo>

File: ur3_gazebo/urdf/ur_with_gripper.xacro (robot description, xacro)
@@ -103,9 +103,9 @@
   </gazebo>
   <!-- Equivalent to the OpenRAVE manipulator denso_robotiq_85_gripper -->
-  <link name="ur3_robotiq_85_gripper" />
+  <link name="ur_gripper_tip_link" />
   <joint name="manipulator_dummy_joint" type="fixed">
     <origin xyz="0 0 0.1441" rpy="0 0 0" />
     <parent link="robotiq_coupler"/>
-    <child link="ur3_robotiq_85_gripper"/>
+    <child link="ur_gripper_tip_link"/>
   </joint>
   <!-- Attach the robotiq 85 gripper -->
@@ -113,14 +113,17 @@
     <origin xyz="0 0 0.004" rpy="0 ${-pi/2} ${pi}"/>
   </xacro:robotiq_85_gripper>
-  <!-- Gazebo FT sensor plugin -->
-  <gazebo reference="wrist_3_link-tool0_fixed_joint">
+  <!-- Gazebo Force/Torque sensor plugin -->
+  <gazebo reference="wrist_3_joint">
     <provideFeedback>true</provideFeedback>
   </gazebo>
+  <!-- <gazebo reference="wrist_3_joint">
+    <preserveFixedJoint>true</preserveFixedJoint>
+  </gazebo> -->
   <gazebo>
     <plugin name="ft_sensor" filename="libgazebo_ros_ft_sensor.so">
-      <updateRate>100.0</updateRate>
+      <updateRate>125.0</updateRate>
       <topicName>ft_sensor/raw</topicName>
       <gaussianNoise>0.0</gaussianNoise>
-      <jointName>wrist_3_link-tool0_fixed_joint</jointName>
+      <jointName>wrist_3_joint</jointName>
     </plugin>
   </gazebo>
