Commit message: Fix connection to real robot with gripper 85

File: ur_pykdl/urdf/ur3.urdf (robot description, URDF)
Before this commit: robot ur3, 22 links, 21 joints
Joints:
- removed joint robotiq_85_left_knuckle_joint
- added joint finger_joint: type revolute, parent robotiq_85_base_link, child robotiq_85_left_knuckle_link, origin xyz=0.05490451627 0.03060114443 0.0 rpy=3.14159265359 0.0 0.0, axis 0 0 1, limit lower=0.0 upper=0.80285 effort=1000 velocity=0.5
- joint robotiq_85_left_finger_tip_joint: mimic joint=robotiq_85_left_knuckle_joint multiplier=-1 -> joint=finger_joint multiplier=-1
- joint robotiq_85_left_inner_knuckle_joint: mimic joint=robotiq_85_left_knuckle_joint offset=0 -> joint=finger_joint offset=0
- joint robotiq_85_right_finger_tip_joint: mimic joint=robotiq_85_left_knuckle_joint multiplier=-1 -> joint=finger_joint multiplier=-1
- joint robotiq_85_right_inner_knuckle_joint: mimic joint=robotiq_85_left_knuckle_joint offset=0 -> joint=finger_joint offset=0
- joint robotiq_85_right_knuckle_joint: mimic joint=robotiq_85_left_knuckle_joint -> joint=finger_joint
