Commit message: Update gripper coupler material

File: ur_gripper_gazebo/urdf/ur_gripper_85.xacro (robot description, xacro)
@@ -78,5 +78,7 @@
         <mesh filename="package://robotiq_description/meshes/robotiq_85_coupler.stl" />
       </geometry>
-      <material name="flat_black"/>
+      <material name="flat_black">
+        <color rgba="0 0 0 1.0"/>
+      </material>
     </visual>
     <collision>

File: ur_gripper_gazebo/urdf/ur_gripper_hande.xacro (robot description, xacro)
@@ -78,5 +78,7 @@
         <mesh filename="package://robotiq_description/meshes/robotiq_85_coupler.stl" />
       </geometry>
-      <material name="flat_black"/>
+      <material name="flat_black">
+        <color rgba="0 0 0 1.0"/>
+      </material>
     </visual>
     <collision>
